Commit message: Collision Information for URDF

File: articubot_ws/src/articubot_description/urdf/common_properties.xacro (robot description, xacro)
@@ -10,3 +10,30 @@
         <color rgba="0.1 0.1 0.1 1" />
     </material>
+    <xacro:macro name="box_inertia" params="m l w h xyz rpy">
+        <inertial>
+            <origin xyz="${xyz}" rpy="${rpy}" />
+            <mass value="${m}" />
+            <inertia ixx="${(m/12) * (h*h + l*l)}" ixy="0" ixz="0"
+                        iyy="${(m/12) * (w*w + l*l)}" iyz="0"
+                        izz="${(m/12) * (w*w + h*h)}" />
+        </inertial>
+    </xacro:macro>
+    <xacro:macro name="cylinder_inertia" params="m r h xyz rpy">
+        <inertial>
+            <origin xyz="${xyz}" rpy="${rpy}" />
+            <mass value="${m}" />
+            <inertia ixx="${(m/12) * (3*r*r + h*h)}" ixy="0" ixz="0"
+                        iyy="${(m/12) * (3*r*r + h*h)}" iyz="0"
+                        izz="${(m/2) * (r*r)}" />
+        </inertial>
+    </xacro:macro>
+    <xacro:macro name="sphere_inertia" params="m r xyz rpy">
+        <inertial>
+            <origin xyz="${xyz}" rpy="${rpy}" />
+            <mass value="${m}" />
+            <inertia ixx="${(2/5) * m * r * r}" ixy="0" ixz="0"
+                        iyy="${(2/5) * m * r * r}" iyz="0"
+                        izz="${(2/5) * m * r * r}" />
+        </inertial>
+    </xacro:macro>
 </robot>

File: articubot_ws/src/articubot_description/urdf/mobile_base.xacro (robot description, xacro)
@@ -4,11 +4,16 @@
     <xacro:property name="base_width" value="0.2794" />
     <xacro:property name="base_height" value="0.1397" />
+    <xacro:property name="base_mass" value="5.0" />
     <xacro:property name="wheel_radius" value="0.034925" />
     <xacro:property name="wheel_length" value="0.0254" />
+    <xacro:property name="wheel_mass" value="1.0" />
     <xacro:property name="lidar_stand_length" value="0.09525" />
     <xacro:property name="lidar_stand_width" value="0.06985" />
     <xacro:property name="lidar_stand_height" value="0.03175" />
+    <xacro:property name="lidar_stand_mass" value="1" />
     <xacro:property name="lidar_length" value="0.0254" />
     <xacro:property name="lidar_radius" value="0.034925" />
+    <xacro:property name="lidar_mass" value="0.5" />
+    <xacro:property name="caster_mass" value="0.5" />
     <!--XARCROs FOR ARTICUBOT-->
     <xacro:macro name="lidar_stand_link">
@@ -21,4 +26,12 @@
                 <material name="black" />
             </visual>
+            <collision>
+                <geometry>
+                    <box size="${lidar_stand_length} ${lidar_stand_width} ${lidar_stand_height}" />
+                </geometry>
+                <origin xyz="0 0 ${lidar_stand_height/2.0}" rpy="0 0 0" />
+            </collision>
+            <xacro:box_inertia m="${lidar_stand_mass}" l="${lidar_stand_length}" w="${lidar_stand_width}" h="${lidar_stand_height}"
+                           xyz="0 0 ${lidar_stand_height / 2.0}" rpy="0 0 0" />
         </link>
     </xacro:macro>
@@ -32,4 +45,12 @@
                 <material name="black" />
             </visual>
+            <collision>
+                <geometry>
+                    <cylinder radius="${lidar_radius}" length="${lidar_length}" />
+                </geometry>
+                <origin xyz="0 0 ${lidar_length/2.0}" rpy="0 0 0" />
+            </collision>
+            <xacro:cylinder_inertia m="${lidar_mass}" r="${lidar_radius}" h="${lidar_length}"
+                             xyz="0 0 0" rpy="0 0 0" />
         </link>
     </xacro:macro>
@@ -43,4 +64,12 @@
                 <material name="grey" />
             </visual>
+            <collision>
+                <geometry>
+                    <cylinder radius="${wheel_radius}" length="${wheel_length}" />
+                </geometry>
+                <origin xyz="0 0 0" rpy="${pi / 2.0} 0 0" />
+            </collision>
+            <xacro:cylinder_inertia m="${wheel_mass}" r="${wheel_radius}" h="${wheel_length}"
+                             xyz="0 0 0" rpy="${pi / 2.0} 0 0" />
         </link>
     </xacro:macro>
@@ -54,4 +83,12 @@
                 <material name="blue" />
             </visual>
+            <collision>
+                <geometry>
+                    <box size="${base_length} ${base_width} ${base_height}" />
+                </geometry>
+                <origin xyz="0 0 ${base_height/2.0}" rpy="0 0 0" />
+            </collision>
+            <xacro:box_inertia m="${base_mass}" l="${base_length}" w="${base_width}" h="${base_height}"
+                           xyz="0 0 ${base_height / 2.0}" rpy="0 0 0" />
         </link>
     </xacro:macro>
@@ -65,4 +102,12 @@
                 <material name="grey" />
             </visual>
+            <collision>
+                <geometry>
+                    <sphere radius="${wheel_radius/2.0}" />
+                </geometry>
+                <origin xyz="0 0 0" rpy="0 0 0" />
+            </collision>
+            <xacro:sphere_inertia m="${caster_mass}" r="${wheel_radius / 2.0}"
+                            xyz="0 0 0" rpy="0 0 0" />
         </link>
     </xacro:macro>
@@ -75,4 +120,5 @@
     <xacro:lidar_link />
     <link name="base_footprint" />
+lidar_mass
     <joint name="base_joint" type="fixed">
         <parent link="base_footprint" />
