Commit message: Made wheels match original articubot

File: articubot_ws/src/articubot_description/urdf/mobile_base.xacro (robot description, xacro)
@@ -61,5 +61,5 @@
                     <cylinder radius="${wheel_radius}" length="${wheel_length}" />
                 </geometry>
-                <origin xyz="0 0 0" rpy="${pi / 2.0} 0 0" />
+                <origin xyz="0 0 0" rpy="0 0 0" />
                 <material name="grey" />
             </visual>
@@ -129,12 +129,12 @@
         <parent link="base_link" />
         <child link="right_wheel_link" />
-        <origin xyz="${-base_length / 4.0} ${-(base_width + wheel_length) / 2.0} 0" rpy="0 0 0" />
-        <axis xyz="0 1 0" />
+        <origin xyz="${-base_length / 4.0} ${-(base_width + wheel_length) / 2.0} 0" rpy="${pi/2} 0 0" />
+        <axis xyz="0 0 -1" />
     </joint>
     <joint name="base_left_wheel_joint" type="continuous">
         <parent link="base_link" />
         <child link="left_wheel_link" />
-        <origin xyz="${-base_length / 4.0} ${(base_width + wheel_length) / 2.0} 0" rpy="0 0 0" />
-        <axis xyz="0 1 0" />
+        <origin xyz="${-base_length / 4.0} ${(base_width + wheel_length) / 2.0} 0" rpy="-${pi/2} 0 0" />
+        <axis xyz="0 0 1" />
     </joint>
     <joint name="base_caster_wheel_joint" type="fixed">

Commit message: Updated masses to reflect actual parts

File: articubot_ws/src/articubot_description/urdf/mobile_base.xacro (robot description, xacro)
@@ -4,16 +4,16 @@
     <xacro:property name="base_width" value="0.2794" />
     <xacro:property name="base_height" value="0.1397" />
-    <xacro:property name="base_mass" value="5.0" />
+    <xacro:property name="base_mass" value="1.4" />
     <xacro:property name="wheel_radius" value="0.034925" />
     <xacro:property name="wheel_length" value="0.0254" />
-    <xacro:property name="wheel_mass" value="1.0" />
+    <xacro:property name="wheel_mass" value="0.03" />
     <xacro:property name="lidar_stand_length" value="0.09525" />
     <xacro:property name="lidar_stand_width" value="0.06985" />
     <xacro:property name="lidar_stand_height" value="0.03175" />
-    <xacro:property name="lidar_stand_mass" value="1" />
+    <xacro:property name="lidar_stand_mass" value="0.06" />
     <xacro:property name="lidar_length" value="0.0254" />
     <xacro:property name="lidar_radius" value="0.034925" />
-    <xacro:property name="lidar_mass" value="0.5" />
-    <xacro:property name="caster_mass" value="0.5" />
+    <xacro:property name="lidar_mass" value="0.12" />
+    <xacro:property name="caster_mass" value="0.04" />
     <!--XARCROs FOR ARTICUBOT-->
     <xacro:macro name="lidar_stand_link">

Commit message: Set up gazebo stuff

File: articubot_ws/src/articubot_description/urdf/mobile_base.xacro (robot description, xacro)
@@ -61,5 +61,5 @@
                     <cylinder radius="${wheel_radius}" length="${wheel_length}" />
                 </geometry>
-                <origin xyz="0 0 0" rpy="0 0 0" />
+                <origin xyz="0 0 0" rpy="${pi / 2.0} 0 0" />
                 <material name="grey" />
             </visual>
@@ -129,12 +129,12 @@
         <parent link="base_link" />
         <child link="right_wheel_link" />
-        <origin xyz="${-base_length / 4.0} ${-(base_width + wheel_length) / 2.0} 0" rpy="${pi/2} 0 0" />
-        <axis xyz="0 0 -1" />
+        <origin xyz="${-base_length / 4.0} ${-(base_width + wheel_length) / 2.0} 0" rpy="0 0 0" />
+        <axis xyz="0 1 0" />
     </joint>
     <joint name="base_left_wheel_joint" type="continuous">
         <parent link="base_link" />
         <child link="left_wheel_link" />
-        <origin xyz="${-base_length / 4.0} ${(base_width + wheel_length) / 2.0} 0" rpy="-${pi/2} 0 0" />
-        <axis xyz="0 0 1" />
+        <origin xyz="${-base_length / 4.0} ${(base_width + wheel_length) / 2.0} 0" rpy="0 0 0" />
+        <axis xyz="0 1 0" />
     </joint>
     <joint name="base_caster_wheel_joint" type="fixed">

File: articubot_ws/src/articubot_description/urdf/my_robot.urdf.xacro (robot description, xacro)
@@ -3,3 +3,4 @@
     <xacro:include filename="common_properties.xacro" />
     <xacro:include filename="mobile_base.xacro" />
+    <xacro:include filename="my_robot.gazebo.xacro"/>
 </robot>

Commit message: Trying this out...?

File: articubot_ws/src/articubot_description/urdf/mobile_base.xacro (robot description, xacro)
@@ -128,5 +128,5 @@
         <parent link="base_link" />
         <child link="right_wheel_link" />
-        <origin xyz="${-base_length / 4.0} ${-(base_width + wheel_length) / 2.0} 0" rpy="0 0 0" />
+        <origin xyz="${-base_length / 4.0} ${-(base_width + wheel_length) / 2.0} 0" rpy="0 0 ${pi}" />
         <axis xyz="0 1 0" />
     </joint>

Commit message: reverting

File: articubot_ws/src/articubot_description/urdf/mobile_base.xacro (robot description, xacro)
@@ -128,5 +128,5 @@
         <parent link="base_link" />
         <child link="right_wheel_link" />
-        <origin xyz="${-base_length / 4.0} ${-(base_width + wheel_length) / 2.0} 0" rpy="0 0 ${pi}" />
+        <origin xyz="${-base_length / 4.0} ${-(base_width + wheel_length) / 2.0} 0" rpy="0 0 0" />
         <axis xyz="0 1 0" />
     </joint>

Commit message: Updated URDF

File: articubot_ws/src/articubot_description/urdf/mobile_base.xacro (robot description, xacro)
@@ -74,6 +74,6 @@
         </link>
     </xacro:macro>
-    <xacro:macro name="base_link">
-        <link name="base_link">
+    <xacro:macro name="chassis">
+        <link name="chassis">
             <visual>
                 <geometry>
@@ -113,5 +113,5 @@
     </xacro:macro>
     <!--INSTANCES OF XACROs-->
-    <xacro:base_link/>
+    <xacro:chassis/>
     <xacro:caster_wheel_link/>
     <xacro:wheel_link prefix="right" />
@@ -119,12 +119,18 @@
     <xacro:lidar_stand_link />
     <xacro:lidar_link />
+    <link name="base_link" />
     <link name="base_footprint" />
-    <joint name="base_joint" type="fixed">
-        <parent link="base_footprint" />
-        <child link="base_link" />
-        <origin xyz="0 0 ${wheel_radius}" rpy="0 0 0"/>
+    <joint name="base_footprint_joint" type="fixed">
+        <parent link="base_link"/>
+        <child link="base_footprint"/>
+        <origin xyz="0 0 0" rpy="0 0 0"/>
+    </joint>
+    <joint name="chassis_joint" type="fixed">
+        <parent link="base_link" />
+        <child link="chassis" />
+        <origin xyz="0 0 0" rpy="0 0 0"/>
     </joint>
     <joint name="base_right_wheel_joint" type="continuous">
-        <parent link="base_link" />
+        <parent link="chassis" />
         <child link="right_wheel_link" />
         <origin xyz="${-base_length / 4.0} ${-(base_width + wheel_length) / 2.0} 0" rpy="0 0 0" />
@@ -132,5 +138,5 @@
     </joint>
     <joint name="base_left_wheel_joint" type="continuous">
-        <parent link="base_link" />
+        <parent link="chassis" />
         <child link="left_wheel_link" />
         <origin xyz="${-base_length / 4.0} ${(base_width + wheel_length) / 2.0} 0" rpy="0 0 0" />
@@ -138,14 +144,14 @@
     </joint>
     <joint name="base_caster_wheel_joint" type="fixed">
-        <parent link="base_link" />
+        <parent link="chassis" />
         <child link="caster_wheel_link" />
         <origin xyz="${base_length / 3.0} 0 ${-wheel_radius / 2.0}" rpy="0 0 0" />
     </joint>
     <joint name="base_lidar_stand_joint" type="fixed">
-        <parent link="base_link" />
+        <parent link="chassis" />
         <child link="lidar_stand_link" />
         <origin xyz="${base_height/2.0} 0 ${base_height}" rpy="0 0 0" />
     </joint>
-    <joint name="lidar_stand_lidar_joint" type="continuous">
+    <joint name="lidar_stand_lidar_joint" type="fixed">
         <parent link="lidar_stand_link" />
         <child link="lidar_link" />

File: articubot_ws/src/articubot_description/urdf/ros2_control.xacro (robot description, xacro)
@@ -7,5 +7,5 @@
             <param name="right_wheel_name">base_right_wheel_joint</param>
             <param name="loop_rate">30</param>
-            <param name="device">/dev/ttyUSB0</param>
+            <param name="device">/dev/serial/by-path/platform-fd500000.pcie-pci-0000:01:00.0-usb-0:1.2:1.0-port0</param>
             <param name="baud_rate">57600</param>
             <param name="timeout_ms">1000</param>
